Commit message: Update

File: quarobo_description/robots/quarobo.urdf.xacro (robot description, xacro)
@@ -5,69 +5,69 @@
     <!-- === body === -->
     <xacro:leg_macro_fi prefix="body" parent="base_link" mesh="body.stl" color="pink">
-        <origin xyz="0 0 0.16505" rpy="0 0 0"/>
+        <origin xyz="0 0 0" rpy="0 0 0"/>
     </xacro:leg_macro_fi>
     <!-- === Front right === -->
-    <xacro:leg_macro_re prefix="FRS" parent="body_link" mesh="front_Shoulder_R.stl" color="green">
-        <origin xyz="-0.027 -0.04905 -0.00075" rpy="0 0 0"/>
+    <xacro:leg_macro_re prefix="FRS" parent="body_link" mesh="FR_Shoulder.stl" color="green">
+        <origin xyz="-0.027 -0.04905 -0.00150" rpy="0 0 0"/>
         <axis xyz="0 1 0"/>
     </xacro:leg_macro_re>
-    <xacro:leg_macro_re prefix="FRL" parent="FRS_link" mesh="front_Leg_R.stl" color="blue">
+    <xacro:leg_macro_re prefix="FRL" parent="FRS_link" mesh="FR_Thigh.stl" color="blue">
         <origin xyz="0 -0.022304 -0.01230" rpy="1.57 0 0"/>
         <axis xyz="1 0 0"/>
     </xacro:leg_macro_re>
-    <xacro:leg_macro_re prefix="FRF" parent="FRL_link" mesh="front_Foot_R.stl" color="purple">
-        <origin xyz="-0.015546 -0.054 0" rpy="0 0 0"/>
+    <xacro:leg_macro_re prefix="FRF" parent="FRL_link" mesh="FR_Shin.stl" color="purple">
+        <origin xyz="-0.01455 -0.054 0" rpy="0 0 0"/>
         <axis xyz="1 0 0"/>
     </xacro:leg_macro_re>
-    <xacro:leg_macro_fi prefix="FRT" parent="FRF_link" mesh="front_Toes_R.stl" color="orange">
-        <origin xyz="-0.003 -0.088 0" rpy="0 0 0"/>
+    <xacro:leg_macro_fi prefix="FRT" parent="FRF_link" mesh="FR_Toe.stl" color="orange">
+        <origin xyz="-0.00550 -0.06800 0" rpy="0 0 0"/>
     </xacro:leg_macro_fi>
     <!-- === Front left === -->
-    <xacro:leg_macro_re prefix="FLS" parent="body_link" mesh="front_Shoulder_L.stl" color="green">
-        <origin xyz="0.027 -0.04905 -0.00075" rpy="0 0 0"/>
+    <xacro:leg_macro_re prefix="FLS" parent="body_link" mesh="FL_Shoulder.stl" color="green">
+        <origin xyz="0.027 -0.04905 -0.00150" rpy="0 0 0"/>
         <axis xyz="0 1 0"/>
     </xacro:leg_macro_re>
-    <xacro:leg_macro_re prefix="FLL" parent="FLS_link" mesh="front_Leg_L.stl" color="blue">
+    <xacro:leg_macro_re prefix="FLL" parent="FLS_link" mesh="FL_Thigh.stl" color="blue">
         <origin xyz="0 -0.022304 -0.01230" rpy="1.57 0 0"/>
         <axis xyz="1 0 0"/>
     </xacro:leg_macro_re>
-    <xacro:leg_macro_re prefix="FLF" parent="FLL_link" mesh="front_Foot_L.stl" color="purple">
-        <origin xyz="0.015546 -0.054 0" rpy="0 0 0"/>
+    <xacro:leg_macro_re prefix="FLF" parent="FLL_link" mesh="FL_Shin.stl" color="purple">
+        <origin xyz="0.01455 -0.054 0" rpy="0 0 0"/>
         <axis xyz="1 0 0"/>
     </xacro:leg_macro_re>
-    <xacro:leg_macro_fi prefix="FLT" parent="FLF_link" mesh="front_Toes_L.stl" color="orange">
-        <origin xyz="0.003 -0.088 0" rpy="0 0 0"/>
+    <xacro:leg_macro_fi prefix="FLT" parent="FLF_link" mesh="FL_Toe.stl" color="orange">
+        <origin xyz="0.00550 -0.06800 0" rpy="0 0 0"/>
     </xacro:leg_macro_fi>
     <!-- === Rear right === -->
-    <xacro:leg_macro_re prefix="RRS" parent="body_link" mesh="rear_Shoulder_R.stl" color="green">
-        <origin xyz="-0.027 0.04905 -0.00075" rpy="0 0 0"/>
+    <xacro:leg_macro_re prefix="RRS" parent="body_link" mesh="RR_Shoulder.stl" color="green">
+        <origin xyz="-0.027 0.04905 -0.00150" rpy="0 0 0"/>
         <axis xyz="0 1 0"/>
     </xacro:leg_macro_re>
-    <xacro:leg_macro_re prefix="RRL" parent="RRS_link" mesh="rear_Leg_R.stl" color="blue">
+    <xacro:leg_macro_re prefix="RRL" parent="RRS_link" mesh="RR_Thigh.stl" color="blue">
         <origin xyz="0 0.022304 -0.01230" rpy="-1.57 0 0"/>
         <axis xyz="1 0 0"/>
     </xacro:leg_macro_re>
-    <xacro:leg_macro_re prefix="RRF" parent="RRL_link" mesh="rear_Foot_R.stl" color="purple">
-        <origin xyz="-0.015546 0.054 0" rpy="0 0 0"/>
+    <xacro:leg_macro_re prefix="RRF" parent="RRL_link" mesh="RR_Shin.stl" color="purple">
+        <origin xyz="-0.01455 0.054 0" rpy="0 0 0"/>
         <axis xyz="1 0 0"/>
     </xacro:leg_macro_re>
-    <xacro:leg_macro_fi prefix="RRT" parent="RRF_link" mesh="rear_Toes_R.stl" color="orange">
-        <origin xyz="-0.003 0.088 0" rpy="0 0 0"/>
+    <xacro:leg_macro_fi prefix="RRT" parent="RRF_link" mesh="RR_Toe.stl" color="orange">
+        <origin xyz="-0.00550 0.06800 0" rpy="0 0 0"/>
     </xacro:leg_macro_fi>
     <!-- === Rear left === -->
-    <xacro:leg_macro_re prefix="RLS" parent="body_link" mesh="rear_Shoulder_L.stl" color="green">
-        <origin xyz="0.027 0.04905 -0.00075" rpy="0 0 0"/>
+    <xacro:leg_macro_re prefix="RLS" parent="body_link" mesh="RL_Shoulder.stl" color="green">
+        <origin xyz="0.027 0.04905 -0.00150" rpy="0 0 0"/>
         <axis xyz="0 1 0"/>
     </xacro:leg_macro_re>
-    <xacro:leg_macro_re prefix="RLL" parent="RLS_link" mesh="rear_Leg_L.stl" color="blue">
+    <xacro:leg_macro_re prefix="RLL" parent="RLS_link" mesh="RL_Thigh.stl" color="blue">
         <origin xyz="0 0.022304 -0.01230" rpy="-1.57 0 0"/>
         <axis xyz="1 0 0"/>
     </xacro:leg_macro_re>
-    <xacro:leg_macro_re prefix="RLF" parent="RLL_link" mesh="rear_Foot_L.stl" color="purple">
-        <origin xyz="0.015546 0.054 0" rpy="0 0 0"/>
+    <xacro:leg_macro_re prefix="RLF" parent="RLL_link" mesh="RL_Shin.stl" color="purple">
+        <origin xyz="0.01455 0.054 0" rpy="0 0 0"/>
         <axis xyz="1 0 0"/>
     </xacro:leg_macro_re>
-    <xacro:leg_macro_fi prefix="RLT" parent="RLF_link" mesh="rear_Toes_L.stl" color="orange">
-        <origin xyz="0.003 0.088 0" rpy="0 0 0"/>
+    <xacro:leg_macro_fi prefix="RLT" parent="RLF_link" mesh="RL_Toe.stl" color="orange">
+        <origin xyz="0.00550 0.06800 0" rpy="0 0 0"/>
     </xacro:leg_macro_fi>
 </robot>

File: quarobo_description/urdf/leg/leg.urdf.xacro (robot description, xacro)
@@ -21,5 +21,5 @@
                 <origin xyz="0 0 0" rpy="0 0 0"/>
                 <geometry>
-                    <mesh filename="package://quarobo_description/meshes/origin_ros_quarobo_stlFiles/${mesh}"/>
+                    <mesh filename="package://quarobo_description/meshes/quarobo_stlFiles/${mesh}"/>
                 </geometry>
                 <material name="${color}"/>
@@ -49,5 +49,5 @@
                 <origin xyz="0 0 0" rpy="0 0 0"/>
                 <geometry>
-                    <mesh filename="package://quarobo_description/meshes/origin_ros_quarobo_stlFiles/${mesh}"/>
+                    <mesh filename="package://quarobo_description/meshes/quarobo_stlFiles/${mesh}"/>
                 </geometry>
                 <material name="${color}"/>
